Commit message: teleoperation node

File: catkin_et/src/finder_description/urdf/finder.xacro (robot description, xacro)
@@ -8,5 +8,5 @@
 <robot name="finder"  xmlns:xacro="http://www.ros.org/wiki/xacro">
 	<!-- Macro para "mandar llamar" a las mallas *.obj -->
-    <xacro:macro name="default_geometry" params="cad_dir:=package://finder_description/meshes_light cad_file extension:=obj">
+    <xacro:macro name="default_geometry" params="cad_dir:=package://finder_description/mallas cad_file extension:=obj">
         <geometry>
 	<!-- Typically, STL/DAE/OBJ model units are in mm, but RViz units are in m, hence models must be scaled down by 1000-->
@@ -93,11 +93,11 @@
 <!--////////////// brazos laterales del chasis ////////////////////-->
 	<!-- brazo frontal derecho chasis -->
-	<xacro:lateral_arms name="right_front_arm" cad_name="brazo_der_frontal_v2" origin="0.3264 0.30255 -0.0629"/>
+	<xacro:lateral_arms name="right_front_arm" cad_name="brazo_der_frontal" origin="0.3264 0.30255 -0.0629"/>
 	<!-- brazo frontal izquierdo chasis -->
-	<xacro:lateral_arms name="left_front_arm" cad_name="brazo_izq_frontal_v2" origin="-0.3264 0.30255 -0.0629"/>
+	<xacro:lateral_arms name="left_front_arm" cad_name="brazo_izq_frontal" origin="-0.3264 0.30255 -0.0629"/>
 	<!-- brazo trasero derecho chasis -->
-	<xacro:lateral_arms name="right_back_arm" cad_name="brazo_der_trasero_v2" origin="0.3264 -0.30255 -0.0629"/>
+	<xacro:lateral_arms name="right_back_arm" cad_name="brazo_der_trasero" origin="0.3264 -0.30255 -0.0629"/>
 	<!-- brazo trasero izquierdo chasis -->
-	<xacro:lateral_arms name="left_back_arm" cad_name="brazo_izq_trasero_v2" origin="-0.3264 -0.30255 -0.0629"/>
+	<xacro:lateral_arms name="left_back_arm" cad_name="brazo_izq_trasero" origin="-0.3264 -0.30255 -0.0629"/>
 <!--///////////////// Brazo 6GDL + Gripper//////////////////-->
 <!--////////////////// "eje tronco" rotation joint //////////////////-->
@@ -151,5 +151,6 @@
 	<link name = "elbow">
 		<visual>
-			<origin xyz= "0 -0.4192 -0.027"/>
+			<!--origin xyz= "0 -0.4192 -0.027"/-->
+			<origin xyz= "0 -0.668 -0.027"/>
 			<xacro:default_geometry cad_file = "codo"/>
 		</visual>

Commit message: gerardo

File: catkin_et/src/finder_description/urdf/finder.xacro (robot description, xacro)
@@ -40,5 +40,5 @@
 	<xacro:macro name = "arms_joints" params="name child origin">
 		<joint name = "${name}" type="revolute">
-			<parent link = "base_link"/>
+			<parent link = "traction"/>
 			<child	link = "${child}"/>
 			<origin xyz ="${origin}"/>
@@ -71,6 +71,6 @@
     </material>
 <!--//////////////////////////  base link //////////////////-->
-	<!--link name = "base_link"></link-->
-	<link name = "base_link">
+	<link name = "base_link"></link>
+	<link name = "traction">
 		<visual>
 			<xacro:default_geometry cad_file = "chasis"/>
@@ -82,4 +82,9 @@
     	</collision>
 	</link>
+	<joint name = "adjustment" type="fixed">
+		<parent link = "base_link"/>
+		<child	link = "traction"/>
+		<origin rpy="0 0 ${pi/2}"/>
+	</joint>
 <!--////////////////// juntas de los brazos laterales del chasis //////////////////-->
 	<!-- junta del brazo frontal derecho -->
@@ -95,13 +100,13 @@
 	<xacro:lateral_arms name="right_front_arm" cad_name="brazo_der_frontal" origin="0.3264 0.30255 -0.0629"/>
 	<!-- brazo frontal izquierdo chasis -->
-	<xacro:lateral_arms name="left_front_arm" cad_name="brazo_izq_frontal" origin="-0.3264 0.30255 -0.0629"/>
+	<xacro:lateral_arms name="left_front_arm" cad_name="brazo_der_frontal" origin="0.3264 0.30255 -0.0629"/>
 	<!-- brazo trasero derecho chasis -->
-	<xacro:lateral_arms name="right_back_arm" cad_name="brazo_der_trasero" origin="0.3264 -0.30255 -0.0629"/>
+	<xacro:lateral_arms name="right_back_arm" cad_name="brazo_der_frontal" origin="0.3264 0.30255 -0.0629"/>
 	<!-- brazo trasero izquierdo chasis -->
-	<xacro:lateral_arms name="left_back_arm" cad_name="brazo_izq_trasero" origin="-0.3264 -0.30255 -0.0629"/>
+	<xacro:lateral_arms name="left_back_arm" cad_name="brazo_der_frontal" origin="0.3264 0.30255 -0.0629"/>
 <!--///////////////// Brazo 6GDL + Gripper//////////////////-->
 <!--////////////////// "eje tronco" rotation joint //////////////////-->
 	<joint name = "base_rotation" type="revolute">
-		<parent link = "base_link"/>
+		<parent link = "traction"/>
 		<child	link = "eje_tronco"/>
 		<origin xyz ="0 -0.30645 ${0.2691-0.0455}" rpy="0 0 0"/>

Commit message: Cambios de cesat

File: catkin_et/src/finder_description/urdf/finder.xacro (robot description, xacro)
@@ -70,6 +70,14 @@
         <color rgba="1.0 1.0 1.0 1.0"/>
     </material>
+<!--//////////////////////////  base footprint //////////////////-->
+	<link name="base_footprint"/>
+	<joint name="base_footprint_joint" type="fixed">
+    	<origin rpy="0 0 0" xyz="0 0 0.04"/>
+    	<!--axis xyz="1 0 0"/-->
+    	<parent link="base_footprint"/>
+    	<child link="base_link"/>
+  </joint>
 <!--//////////////////////////  base link //////////////////-->
-	<link name = "base_link"></link>
+	<link name = "base_link"/>
 	<link name = "traction">
 		<visual>

Commit message: Código de César

File: catkin_et/src/finder_description/urdf/finder.xacro (robot description, xacro)
@@ -70,12 +70,4 @@
         <color rgba="1.0 1.0 1.0 1.0"/>
     </material>
-<!--//////////////////////////  base footprint //////////////////-->
-	<link name="base_footprint"/>
-	<joint name="base_footprint_joint" type="fixed">
-    	<origin rpy="0 0 0" xyz="0 0 0.04"/>
-    	<!--axis xyz="1 0 0"/-->
-    	<parent link="base_footprint"/>
-    	<child link="base_link"/>
-  </joint>
 <!--//////////////////////////  base link //////////////////-->
 	<link name = "base_link"/>
@@ -90,4 +82,5 @@
     	</collision>
 	</link>
+	<!--Esta transformacion se hace para que los datos del SLAM correspondan a la correcta orientacion del robot-->
 	<joint name = "adjustment" type="fixed">
 		<parent link = "base_link"/>
